File: hardware/GlucoBit-v2/GlucoBit-v2.kicad_pcb (KiCad board)
At the start: 4 copper layers, 55 x 30.4 mm, 43 parts, among them J1 USB-C-P16, J2 B2B-PH-K-S, J3 Conn_01x02_Socket, J6 B2B-PH-K-S, SW1 RESET, SW2 BOOT, U1 ESP32-S3-WROOM-1-N8, U2 BQ24040DSQR, U3 TLV75801PDBV, U4 ESD7104MUTAG, U5 MAX98357AETE+T, U6 08JQ-BT

Commit message: Update PCB after DFM
Parts:
- U4: value ESD7104MUTAG -> USBLC6-2SC6; footprint GlucoBit v2:IC_ESD7104MUTAG -> GlucoBit v2:SOT95P280X145-6N
- moved U4 8.17 mm to (72.2, 49.5), turned to 90 degrees
- moved C4 7.53 mm to (79.8, 50.9), turned to 90 degrees
- moved R3 6.89 mm to (81.5, 55.6), turned to -90 degrees
- moved R2 5.81 mm to (81.5, 52.3), turned to -90 degrees
- moved U2 4.99 mm to (74.2, 54.8)
- moved C5 4.07 mm to (72.0, 59.2)
- moved R4 4.06 mm to (75.8, 48.0)
- moved R6 3.95 mm to (74.7, 65.3)
- moved C1 3.91 mm to (76.8, 51.0)
- moved U3 3.90 mm to (78.4, 54.5), turned to 0 degrees
- moved C2 3.40 mm to (74.0, 59.2)
- moved C3 2.86 mm to (76.7, 58.0)
- moved R10 2.65 mm to (80.2, 59.0)
- moved R16 2.60 mm to (80.6, 61.6), turned to 90 degrees
- moved R5 2.49 mm to (76.3, 65.3)
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Connections:
- J1 pad A6: USB_P -> /USB_D+
- J1 pad A7: USB_N -> /USB_D-
- J1 pad B6: USB_P -> /USB_D+
- J1 pad B7: USB_N -> /USB_D-
- U1 pad 10: CH -> LRCLK
- U1 pad 11: PGOOD -> DIN
- U1 pad 12: PER -> BCLK
- U1 pad 13: USB_N -> /USB_N
- U1 pad 14: USB_P -> /USB_P
- U1 pad 18: CS -> LED
- U1 pad 19: MOSI -> BL
- U1 pad 20: CLK -> RST
- U1 pad 22: RST -> CS
- U1 pad 23: unconnected-(U1-IO21-Pad23) -> CLK
- U1 pad 24: unconnected-(U1-IO47-Pad24) -> MOSI
- U1 pad 25: unconnected-(U1-IO48-Pad25) -> CH
- U1 pad 26: unconnected-(U1-IO45-Pad26) -> PGOOD
- U1 pad 34: unconnected-(U1-IO41-Pad34) -> PER
- U1 pad 4: BCLK -> unconnected-(U1-IO4-Pad4)
- U1 pad 5: LRCLK -> unconnected-(U1-IO5-Pad5)
- U1 pad 6: DIN -> unconnected-(U1-IO6-Pad6)
- U1 pad 8: BL -> unconnected-(U1-IO15-Pad8)
- U1 pad 9: LED -> unconnected-(U1-IO16-Pad9)
- U2 pad V: (no net) -> GND
- U4 pad 1: USB_N -> /USB_D-
- U4 pad 2: USB_P -> GND
- U4 pad 3: GND -> /USB_D+
- U4 pad 4: /5VIN -> /USB_P
- U4 pad 5: unconnected-(U4-I/O_5-Pad5) -> /5VIN
- U4 pad 6: unconnected-(U4-Pad6) -> /USB_N
Routing:
- net +3V3: track 0.00 -> 105.4 mm, vias 0 -> 6
- net ENABLE: track 0.00 -> 82.5 mm, vias 0 -> 2
- net /VOUT: track 0.00 -> 65.4 mm, vias 0 -> 1
- net Net-(U5-OUTP): track 0.00 -> 55.4 mm, vias 0 -> 2
- net Net-(U5-OUTN): track 0.00 -> 48.6 mm, vias 0 -> 2
- net BOOT: track 0.00 -> 44.6 mm, vias 0 -> 2
- net GND: track 24.4 -> 66.5 mm, vias 0 -> 68
- net DIN: track 0.00 -> 38.3 mm
- net BCLK: track 0.00 -> 34.5 mm, vias 0 -> 2
- net PGOOD: track 0.00 -> 32.4 mm, vias 0 -> 3
- net LRCLK: track 0.00 -> 32.2 mm, vias 0 -> 2
- net CH: track 0.00 -> 30.9 mm, vias 0 -> 3
- net Touch: track 0.00 -> 29.2 mm, vias 0 -> 1
- net /USB_N: track 0.00 -> 25.8 mm
- net /USB_P: track 0.00 -> 23.9 mm
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- added copper zone on In2.Cu, net /5VIN
- added copper zone on B.Cu, net GND
- added copper zone on F.Cu, net GND
- added copper zone on In1.Cu, net GND
