File: hardware/GlucoBit-v2/GlucoBit-v2.kicad_sch (KiCad schematic)
At the start: 43 parts, among them J1 USB-C-P16, J2 B2B-PH-K-S, J3 Conn_01x02_Socket, J6 B2B-PH-K-S, SW1 RESET, SW2 BOOT, U1 ESP32-S3-WROOM-1-N8, U2 BQ24040DSQR, U3 TLV75801PDBV, U4 ESD7104MUTAG, U5 MAX98357AETE+T, U6 08JQ-BT

Commit message: Update PCB after DFM
Parts:
- removed U4: ESD7104MUTAG, GlucoBit v2:IC_ESD7104MUTAG, symbol GlucoBit v2:ESD7104MUTAG
- added U4: USBLC6-2SC6, GlucoBit v2:SOT95P280X145-6N, symbol GlucoBit v2:USBLC6-2SC6
Connections:
- net 5VIN: now also U4.5
- net BCLK: now also U1.12 (IO8); no longer U1.4 (IO4)
- net BL: now also U1.19 (IO11); no longer U1.8 (IO15)
- net CH: now also U1.25 (IO48); no longer U1.10 (IO17)
- net CLK: now also U1.23 (IO21); no longer U1.20 (IO12)
- net CS: now also U1.22 (IO14); no longer U1.18 (IO10)
- net DIN: now also U1.11 (IO18); no longer U1.6 (IO6)
- net GND: now also U4.2
- net LED: now also U1.18 (IO10); no longer U1.9 (IO16)
- net LRCLK: now also U1.10 (IO17); no longer U1.5 (IO5)
- net MOSI: now also U1.24 (IO47); no longer U1.19 (IO11)
- net PER: now also U1.34 (IO41); no longer U1.12 (IO8)
- net PGOOD: now also U1.26 (IO45); no longer U1.11 (IO18)
- net RST: now also U1.20 (IO12); no longer U1.22 (IO14)
- net USB_N: now also U4.6; no longer J1.A7 (DN1), J1.B7 (DN2)
- net USB_P: now also U4.4; no longer J1.A6 (DP1), J1.B6 (DP2)
- new net USB_D+: J1.A6 (DP1), J1.B6 (DP2), U4.3
- new net USB_D-: J1.A7 (DN1), J1.B7 (DN2), U4.1
- no-connect marks 25 -> 23

Commit message: Update UI
Parts:
- added D4: LED, LED_SMD:LED_0805_2012Metric, symbol Device:LED
- added V1: 2.2, symbol Simulation_SPICE:VDC
Connections:
- new net: D4.1 (K), V1.2
- new net: D4.2 (A), V1.1
Changed lines of the file:
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@@
 	(wire
 		(pts
+			(xy 106.68 25.4) (xy 106.68 26.67)
+		)
+		(stroke
+			(width 0)
+			(type default)
+		)
+	)
+	(wire
+		(pts
 			(xy 234.95 162.56) (xy 246.38 162.56)
 		)
@@
 	(wire
 		(pts
+			(xy 106.68 34.29) (xy 106.68 35.56)
+		)
+		(stroke
+			(width 0)
+			(type default)
+		)
+	)
+	(wire
+		(pts
 			(xy 306.07 63.5) (xy 306.07 66.04)
 		)
@@
 	(wire
 		(pts
+			(xy 93.98 35.56) (xy 106.68 35.56)
+		)
+		(stroke
+			(width 0)
+			(type default)
+		)
+	)
+	(wire
+		(pts
 			(xy 106.68 185.42) (xy 106.68 186.69)
 		)
@@
 	(wire
 		(pts
+			(xy 93.98 25.4) (xy 106.68 25.4)
+		)
+		(stroke
+			(width 0)
+			(type default)
+		)
+	)
+	(wire
+		(pts
 			(xy 50.8 31.75) (xy 68.58 31.75)
 		)
@@
 	)
 	(symbol
+		(lib_id "Device:LED")
+		(at 106.68 30.48 90)
+		(unit 1)
+		(exclude_from_sim no)
+		(in_bom yes)
+		(on_board yes)
+		(dnp no)
+		(fields_autoplaced yes)
+		(property "Reference" "D4"
+			(at 110.49 30.7974 90)
+			(effects
+				(font
+					(size 1.27 1.27)
+				)
+				(justify right)
+			)
+		)
+		(property "Value" "LED"
+			(at 110.49 33.3374 90)
+			(effects
+				(font
+					(size 1.27 1.27)
+				)
+				(justify right)
+			)
+		)
+		(property "Footprint" "LED_SMD:LED_0805_2012Metric"
+			(at 106.68 30.48 0)
+			(effects
+				(font
+					(size 1.27 1.27)
+				)
+				(hide yes)
+			)
+		)
+		(property "Datasheet" "~"
+			(at 106.68 30.48 0)
+			(effects
+				(font
+					(size 1.27 1.27)
+				)
+				(hide yes)
+			)
+		)
+		(property "Description" "Light emitting diode"
+			(at 106.68 30.48 0)
+			(effects
+				(font
+					(size 1.27 1.27)
+				)
+				(hide yes)
+			)
+		)
+		(property "Sim.Pins" "1=K 2=A"
+			(at 106.68 30.48 0)
+			(effects
+				(font
+					(size 1.27 1.27)
+				)
+				(hide yes)
+			)
+		)
+		(pin "2"
+		)
+		(pin "1"
+		)
+		(instances
+			(project "GlucoBit-v2"
+				(path "/f630bb66-a5b1-4223-898d-4f58907e4cf3"
+					(reference "D4")
+					(unit 1)
+				)
+			)
+		)
+	)
+	(symbol
 		(lib_id "power:+3V3")
 		(at 50.8 157.48 0)
@@
 					(unit 1)
 				)
+			)
+		)
+	)
+	(symbol
+		(lib_id "Simulation_SPICE:VDC")
+		(at 93.98 30.48 0)
+		(unit 1)
+		(exclude_from_sim no)
+		(in_bom yes)
+		(on_board yes)
+		(dnp no)
+		(fields_autoplaced yes)
+		(property "Reference" "V1"
+			(at 97.79 29.0801 0)
+			(effects
+				(font
+					(size 1.27 1.27)
+				)
+				(justify left)
+			)
+		)
+		(property "Value" "2.2"
+			(at 97.79 31.6201 0)
+			(effects
+				(font
+					(size 1.27 1.27)
+				)
+				(justify left)
+			)
+		)
+		(property "Footprint" ""
+			(at 93.98 30.48 0)
+			(effects
+				(font
+					(size 1.27 1.27)
+				)
+				(hide yes)
+			)
+		)
+		(property "Datasheet" "https://ngspice.sourceforge.io/docs/ngspice-html-manual/manual.xhtml#sec_Independent_Sources_for"
+			(at 93.98 30.48 0)
+			(effects
+				(font
+					(size 1.27 1.27)
+				)
+				(hide yes)
+			)
+		)
+		(property "Description" "Voltage source, DC"
+			(at 93.98 30.48 0)
+			(effects
+				(font
+					(size 1.27 1.27)
+				)
+				(hide yes)
+			)
+		)
+		(property "Sim.Pins" "1=+ 2=-"
+			(at 93.98 30.48 0)
+			(effects
+				(font
+					(size 1.27 1.27)
+				)
+				(hide yes)
+			)
+		)
+		(property "Sim.Type" "DC"
+			(at 93.98 30.48 0)
+			(effects
+				(font
+					(size 1.27 1.27)
+				)
+				(hide yes)
+			)
+		)
+		(property "Sim.Device" "V"
+			(at 93.98 30.48 0)
+			(effects
+				(font
+					(size 1.27 1.27)
+				)
+				(justify left)
+				(hide yes)
+			)
+		)
+		(pin "2"
+		)
+		(pin "1"
+		)
+		(instances
+			(project ""
+				(path "/f630bb66-a5b1-4223-898d-4f58907e4cf3"
+					(reference "V1")
+					(unit 1)
+				)
